File: Crystal-Zeliska-back.kicad_pcb (KiCad board)
At the start: 2 copper layers, 183.5 x 114.3 mm, 127 parts, among them K1 KEYSW, K10 KEYSW, K11 KEYSW, K12 KEYSW, K13 KEYSW, K14 KEYSW, K15 KEYSW, K16 KEYSW, K17 KEYSW, K18 KEYSW, K19 KEYSW, K2 KEYSW, K20 KEYSW, K21 KEYSW, K22 KEYSW, K23 KEYSW, K24 KEYSW, K25 KEYSW, K26 KEYSW, K27 KEYSW, K28 KEYSW, K29 KEYSW, K3 KEYSW, K30 KEYSW, K31 KEYSW, K4 KEYSW, K5 KEYSW, K6 KEYSW, K7 KEYSW, K8 KEYSW, K9 KEYSW, SW1 SW_Push_Open_Dual, U1 ProMicro, U2 TRRS

Commit message: Second commit, updated plate,pcb,bottom, cleaned file etc
Parts:
- moved SW1 8.52 mm to (210.3, 97.5)
- moved SW1 8.52 mm to (208.9, 97.5)
Connections:
- net /+5V renamed +5V
- net /GND renamed GND
- net /RST renamed RST
- net /SCL-OLED renamed SCL-OLED
- net /SDA-OLED renamed SDA-OLED
- net /TRRS1 renamed TRRS1
- net /col0 renamed Col0
- net /col1 renamed Col1
- net /col2 renamed Col2
- net /col3 renamed Col3
- net /col4 renamed Col4
- net /col5 renamed Col5
- net /col6 renamed Col6
- net /ledin renamed ledin
- net /row0 renamed Row0
- net /row1 renamed Row1
- net /row2 renamed Row2
- net /row3 renamed Row3
- net /row4 renamed Row4
Routing:
- net RST: track 64.6 -> 91.0 mm
- net GND: track 609.0 -> 629.0 mm
