File: Crystal-Zeliska-plate.kicad_pcb (KiCad board)
At the start: 2 copper layers, 0 parts

Commit message: Second commit, updated plate,pcb,bottom, cleaned file etc
Other:
- board outline added: 182.6 x 114.3 mm
