File: Crystal-Zeliska.sch (KiCad schematic (older format))
At the start: 74 parts, among them K1 KEYSW, K10 KEYSW, K11 KEYSW, K12 KEYSW, K13 KEYSW, K14 KEYSW, K15 KEYSW, K16 KEYSW, K17 KEYSW, K18 KEYSW, K19 KEYSW, K2 KEYSW, K20 KEYSW, K21 KEYSW, K22 KEYSW, K23 KEYSW, K24 KEYSW, K25 KEYSW, K26 KEYSW, K27 KEYSW, K28 KEYSW, K29 KEYSW, K3 KEYSW, K30 KEYSW, K31 KEYSW, K4 KEYSW, K5 KEYSW, K6 KEYSW, K7 KEYSW, K8 KEYSW, K9 KEYSW, SW1 SW_Push_Open_Dual, U1 ProMicro, U2 TRRS

Commit message: Second commit, updated plate,pcb,bottom, cleaned file etc
Connections:
- net col0 renamed Col0
- net col1 renamed Col1
- net col2 renamed Col2
- net col3 renamed Col3
- net col4 renamed Col4
- net col5 renamed Col5
- net col6 renamed Col6
- net row0 renamed Row0
- net row1 renamed Row1
- net row2 renamed Row2
- net row3 renamed Row3
- net row4 renamed Row4
Other:
- moved on the sheet: Brd1, D35, D37, D38, D39, D40, D41, D42, D43, SW1, U2

Commit message: updated Gerber
Parts:
- added R1: 10k, Keebio-Parts:Resistor-Hybrid, symbol Device:R
Connections:
- net +5V: now also R1.1
- net RST: now also R1.2
Changed lines of the file:
@@
 RST
 Wire Wire Line
-	4500 1900 4700 1900
+	4500 1900 4600 1900
 Text GLabel 4500 1900 0    50   Input ~ 0
 RST
@@
 Text GLabel 1700 1650 0    50   Input ~ 0
 GND
+$Comp
+L Device:R R1
+U 1 1 6072FBE5
+P 4900 1600
+F 0 "R1" V 4693 1600 50  0000 C CNN
+F 1 "10k" V 4784 1600 50  0000 C CNN
+F 2 "Keebio-Parts:Resistor-Hybrid" V 4830 1600 50  0001 C CNN
+F 3 "~" H 4900 1600 50  0001 C CNN
+	1    4900 1600
+	0    1    1    0
+$EndComp
+Wire Wire Line
+	4750 1600 4600 1600
+Wire Wire Line
+	4600 1600 4600 1900
+Connection ~ 4600 1900
+Wire Wire Line
+	4600 1900 4700 1900
+Wire Wire Line
+	5050 1600 5200 1600
+Text GLabel 5200 1600 2    50   Input ~ 0
++5V
 $EndSCHEMATC
